Commit message: corrected the joints' names.

File: robots/sunflower1_1.xacro (robot description, xacro)
@@ -105,5 +105,5 @@
 		</link>
 		<xacro:ax12 name="${name}_lower" parent="${name}" minPosition="-1.5707" maxPosition="1.5707" maxVelocity="1">
-			<origin rpy="0 0 1.57079" xyz="0 0 0" />
+			<origin rpy="0 0 -1.57079" xyz="0 0 0" />
 		</xacro:ax12>
 		<xacro:fp04_02 name="${name}_lower_hinge" parent="${name}_lower">
@@ -117,8 +117,8 @@
 			<origin rpy="0 0 -1.57079" xyz="0 0 0" />
 		</xacro:ax12inverted>
-		<xacro:ax12 name="head_tilt" parent="head_pan" minPosition="-1.5707" maxPosition="1.5707" maxVelocity="1">
-			<origin rpy="0 0 0" xyz="0 0 0" />
+		<xacro:ax12 name="head_roll" parent="head_pan" minPosition="-1.5707" maxPosition="1.5707" maxVelocity="1">
+			<origin rpy="0 0 3.142" xyz="0 0 0" />
 		</xacro:ax12>
-		<xacro:fp04_02 name="head_tilt_hinge" parent="head_tilt">
+		<xacro:fp04_02 name="head_roll_hinge" parent="head_roll">
 		</xacro:fp04_02>
 	</xacro:macro>
@@ -405,5 +405,5 @@
 		<origin rpy="0 0 0" xyz="0 0 0" />
 	</xacro:neck>
-	<xacro:head name="head" parent="head_tilt_hinge">
+	<xacro:head name="head" parent="head_roll_hinge">
 		<origin rpy="0 0 0" xyz="0 0 0" />
 	</xacro:head>
