Commit message: set pioneer caster joint as fixed, and create a joint state publisher with GUI for checking the urdf

File: robots/pioneer3dx.urdf.xacro (robot description, xacro)
@@ -121,5 +121,5 @@
 	</joint>
 	<!-- Caster -->
-	<joint name="base_caster_swivel_joint" type="continuous">
+	<joint name="base_caster_swivel_joint" type="fixed">
 		<origin xyz="-0.180 0 0.055" rpy="0 0 0"/>
         <axis xyz="0 0 1" />
@@ -137,19 +137,19 @@
 				 iyy="0.01" iyz="0" izz="0.01"/>
   	 	</inertial>
-	<visual name="pioneer_geom">
-		<origin xyz="-0.004 0 0" rpy="0 0 0"/>
-		<geometry name="pioneer_geom">
-			<mesh filename="package://sf_description/meshes/p3dx_meshes/caster_swivel.stl"/>
-		</geometry>
-		<material name="caster_swivel">
-			<color rgba="0.5 0.5 0.5 1"/>
-		</material>
-	</visual>
-	<collision>
-		<origin xyz="0 0 0" rpy="0 0 0"/>
-		<geometry>
-			<box size="0 0 0"/>
-		</geometry>
-	</collision>
+	    <visual name="pioneer_geom">
+		    <origin xyz="-0.004 0 0" rpy="0 0 0"/>
+		    <geometry name="pioneer_geom">
+	    		<mesh filename="package://sf_description/meshes/p3dx_meshes/caster_swivel.stl"/>
+    		</geometry>
+		    <material name="caster_swivel">
+			    <color rgba="0.5 0.5 0.5 1"/>
+    		</material>
+	    </visual>
+    	<collision>
+	    	<origin xyz="0 0 0" rpy="0 0 0"/>
+	    	<geometry>
+	    		<box size="0 0 0"/>
+	    	</geometry>
+	    </collision>
 	</link>
 	<gazebo reference="caster_swivel">
@@ -164,30 +164,30 @@
 				 iyy="0.015218160428" iyz="-0.000004273467" izz="0.011763977943"/>
   	 	</inertial>
-	<visual name="pioneer_geom">
-		<origin xyz="0 0 0" rpy="0 0 0"/>
-		<geometry name="pioneer_geom">
-			<mesh filename="package://sf_description/meshes/p3dx_meshes/caster_hubcap.stl"/>
-		</geometry>
-		<material name="caster_swivel">
-			<color rgba="0.5 0.5 0.5 1"/>
-		</material>
-	</visual>
-	<collision>
-		<origin xyz="0 0 0" rpy="0 0 0"/>
-		<geometry>
-			<box size="0.05 0.05 0.05"/>
-		</geometry>
-	</collision>
+    	<visual name="pioneer_geom">
+	    	<origin xyz="0 0 0" rpy="0 0 0"/>
+	    	<geometry name="pioneer_geom">
+	    		<mesh filename="package://sf_description/meshes/p3dx_meshes/caster_hubcap.stl"/>
+	    	</geometry>
+	    	<material name="caster_swivel">
+	    		<color rgba="0.5 0.5 0.5 1"/>
+	    	</material>
+	    </visual>
+    	<collision>
+	    	<origin xyz="0 0 0" rpy="0 0 0"/>
+	    	<geometry>
+	    		<box size="0.05 0.05 0.05"/>
+	    	</geometry>
+	    </collision>
 	</link>
 	<gazebo reference="caster_hubcap">
 		<material value="Gazebo/Grey"/>
 	</gazebo>
-	<joint name="caster_swivel_hubcap_joint" type="continuous">
+	<joint name="caster_swivel_hubcap_joint" type="fixed">
 		<origin xyz="-0.026 0 -0.016" rpy="0 0 0"/>
 		<axis xyz="0 1 0"/>
 		<anchor xyz="0 0 0"/>
-    <limit effort="100" velocity="100" k_velocity="0" />
-    <joint_properties damping="0.0" friction="0.0" />
-	  <parent link="caster_swivel"/>
+        <limit effort="100" velocity="100" k_velocity="0" />
+        <joint_properties damping="0.0" friction="0.0" />
+	    <parent link="caster_swivel"/>
 		<child link="caster_wheel"/>
 	</joint>
@@ -199,20 +199,20 @@
 				 iyy="0.015218160428" iyz="-0.000004273467" izz="0.011763977943"/>
   	 	</inertial>
-	<visual name="pioneer_geom">
-		<origin xyz="0 0 0" rpy="0 0 0"/>
-		<geometry name="pioneer_geom">
-			<mesh filename="package://sf_description/meshes/p3dx_meshes/caster_wheel.stl"/>
-		</geometry>
-		<material name="WheelBlack">
-			<color rgba="0.117 0.117 0.117 1"/>
-		</material>
-	</visual>
-	<collision>
-		<origin xyz="0 0 0" rpy="${-3.1415927/2.0} 0 0"/>
-		<geometry>
+	    <visual name="pioneer_geom">
+		    <origin xyz="0 0 0" rpy="0 0 0"/>
+		    <geometry name="pioneer_geom">
+		    	<mesh filename="package://sf_description/meshes/p3dx_meshes/caster_wheel.stl"/>
+		    </geometry>
+		    <material name="WheelBlack">
+		    	<color rgba="0.117 0.117 0.117 1"/>
+		    </material>
+	    </visual>
+	    <collision>
+		    <origin xyz="0 0 0" rpy="${-3.1415927/2.0} 0 0"/>
+		    <geometry>
 			<!--<mesh filename="package://sf_description/meshes/p3dx_meshes/caster_wheel.stl"/>-->
-			<cylinder radius="0.0375" length="0.01"/>
-		</geometry>
-	</collision>
+		    	<cylinder radius="0.0375" length="0.01"/>
+		    </geometry>
+	    </collision>
 	</link>
 	<gazebo reference="left_hub">
@@ -278,10 +278,10 @@
 		</visual>
 		<collision>
-		<origin xyz="0 0 0" rpy="${-3.1415927/2.0} 0 0"/>
-		<geometry>
+	    	<origin xyz="0 0 0" rpy="${-3.1415927/2.0} 0 0"/>
+	    	<geometry>
 			<!--<mesh filename="package://sf_description/meshes/p3dx_meshes/caster_wheel.stl"/>-->
-			<cylinder radius="0.09" length="0.01"/>
-		</geometry>
-	</collision>
+	    		<cylinder radius="0.09" length="0.01"/>
+	    	</geometry>
+	    </collision>
 	</link>
 	<gazebo reference="right_hub">
